Commit message: Fixed gravity bug for gripper in Gazebo; Fixed vertical bug when gravity pulls gripper to open in vertical position

File: src/robotiq_85/robotiq_description/urdf/robotiq_85_gripper.gazebo.xacro (robot description, xacro)
@@ -5,5 +5,5 @@
         <xacro:macro name="hand_gazebo" params="link">
             <gazebo reference="${link}">
-                <material>Gazebo/Black</material>
+                <material>Gazebo/DarkGrey</material>
                 <!-- <mu1>0.2</mu1> -->
                 <!-- <mu2>0.2</mu2> -->

File: src/robotiq_85/robotiq_description/urdf/robotiq_85_gripper.transmission.xacro (robot description, xacro)
@@ -17,12 +17,24 @@
                 <joint>${prefix}robotiq_85_left_knuckle_joint</joint>
                 <mimicJoint>${prefix}robotiq_85_right_knuckle_joint</mimicJoint>
+                <multiplier>1.0</multiplier>
+                <offset>0.0</offset>
+                <maxEffort>1000</maxEffort> <!-- This is crucial -->
+                <hasPID/> <!-- This is crucial -->
             </plugin>
             <plugin filename="libroboticsgroup_upatras_gazebo_mimic_joint_plugin.so" name="${prefix}mimic_robotiq_85_2">
                 <joint>${prefix}robotiq_85_left_knuckle_joint</joint>
                 <mimicJoint>${prefix}robotiq_85_left_inner_knuckle_joint</mimicJoint>
+                <multiplier>1.0</multiplier>
+                <offset>0.0</offset>
+                <maxEffort>0.1</maxEffort> <!-- This is crucial -->
+                <hasPID/> <!-- This is crucial -->
             </plugin>
             <plugin filename="libroboticsgroup_upatras_gazebo_mimic_joint_plugin.so" name="${prefix}mimic_robotiq_85_3">
                 <joint>${prefix}robotiq_85_left_knuckle_joint</joint>
                 <mimicJoint>${prefix}robotiq_85_right_inner_knuckle_joint</mimicJoint>
+                <multiplier>1.0</multiplier>
+                <offset>0.0</offset>
+                <maxEffort>0.1</maxEffort> <!-- This is crucial -->
+                <hasPID/> <!-- This is crucial -->
             </plugin>
             <plugin filename="libroboticsgroup_upatras_gazebo_mimic_joint_plugin.so" name="${prefix}mimic_robotiq_85_4">
@@ -30,5 +42,7 @@
                 <mimicJoint>${prefix}robotiq_85_left_finger_tip_joint</mimicJoint>
                 <multiplier>-1.0</multiplier>
-                <!-- <offset>0.0</offset> -->
+                <offset>0.0</offset>
+                <maxEffort>0.1</maxEffort> <!-- This is crucial -->
+                <hasPID/> <!-- This is crucial -->
             </plugin>
             <plugin filename="libroboticsgroup_upatras_gazebo_mimic_joint_plugin.so" name="${prefix}mimic_robotiq_85_5">
@@ -36,6 +50,11 @@
                 <mimicJoint>${prefix}robotiq_85_right_finger_tip_joint</mimicJoint>
                 <multiplier>-1.0</multiplier>
-                <!-- <offset>0.0</offset> -->
+                <offset>0.0</offset>
+                <maxEffort>0.1</maxEffort> <!-- This is crucial -->
+                <hasPID/> <!-- This is crucial -->
             </plugin>
+            <!-- This plugin fixes the problem when the object slips from the gripper
+                by "fixing" the object to the gripper
+            -->
             <!-- <plugin name="gazebo_grasp_fix" filename="libgazebo_grasp_fix.so">
                 <arm>

File: src/robotiq_85/robotiq_description/urdf/robotiq_85_gripper.urdf.xacro (robot description, xacro)
@@ -41,5 +41,5 @@
       <origin rpy="0.0 0.0 0.0" xyz="0.05490451627 -0.03060114443 0.0"/>
       <limit lower="-3.14" upper="3.14" velocity="100.0" effort="1000"/>
-      <mimic joint="${prefix}robotiq_85_left_knuckle_joint"/>
+      <!-- <mimic joint="${prefix}robotiq_85_left_knuckle_joint"/> -->
     </joint>
     <link name="${prefix}robotiq_85_left_knuckle_link">
@@ -134,6 +134,6 @@
       <axis xyz="0 0 1"/>
       <origin xyz="0.06142 0.0127 0" rpy="${pi} 0.0 0.0" />
-      <limit lower="-3.14" upper="3.14" velocity="100.0" effort="0.1"/>
-      <mimic joint="${prefix}robotiq_85_left_knuckle_joint" offset="0"/>
+      <limit lower="-3.14" upper="3.14" velocity="100.0" effort="1000"/>
+      <!-- <mimic joint="${prefix}robotiq_85_left_knuckle_joint" offset="0"/> -->
     </joint>
     <joint name="${prefix}robotiq_85_right_inner_knuckle_joint" type="continuous">
@@ -142,6 +142,6 @@
       <axis xyz="0 0 1"/>
       <origin xyz="0.06142 -0.0127 0" rpy="0 0 0"/>
-      <limit lower="-3.14" upper="3.14" velocity="100.0" effort="0.1"/>
-      <mimic joint="${prefix}robotiq_85_left_knuckle_joint" offset="0"/>
+      <limit lower="-3.14" upper="3.14" velocity="100.0" effort="1000"/>
+      <!-- <mimic joint="${prefix}robotiq_85_left_knuckle_joint" offset="0"/> -->
     </joint>
     <link name="${prefix}robotiq_85_left_inner_knuckle_link">
@@ -188,6 +188,6 @@
       <axis xyz="0 0 1"/>
       <origin xyz="0.04303959807 -0.03759940821 0.0" rpy="0.0 0.0 0.0"/>
-      <limit lower="-3.14" upper="3.14" velocity="100.0" effort="0.1"/>
-      <mimic joint="${prefix}robotiq_85_left_knuckle_joint" multiplier="-1"/>
+      <limit lower="-3.14" upper="3.14" velocity="100.0" effort="1000"/>
+      <!-- <mimic joint="${prefix}robotiq_85_left_knuckle_joint" multiplier="-1"/> -->
     </joint>
     <joint name="${prefix}robotiq_85_right_finger_tip_joint" type="continuous">
@@ -196,6 +196,6 @@
       <axis xyz="0 0 1"/>
       <origin rpy="0.0 0.0 0.0" xyz="0.04303959807 -0.03759940821  0.0"/>
-      <limit lower="-3.14" upper="3.14" velocity="100.0" effort="0.1"/>
-      <mimic joint="${prefix}robotiq_85_left_knuckle_joint" multiplier="-1"/>
+      <limit lower="-3.14" upper="3.14" velocity="100.0" effort="1000"/>
+      <!-- <mimic joint="${prefix}robotiq_85_left_knuckle_joint" multiplier="-1"/> -->
     </joint>
     <link name="${prefix}robotiq_85_left_finger_tip_link">

File: src/ur5/ur5_description/urdf/ur5_robotiq85_gripper.urdf.xacro (robot description, xacro)
@@ -35,5 +35,5 @@
     <mu1>0.9</mu1>
     <mu2>0.9</mu2>
-    <material>Gazebo/FlatBlack</material>
+    <material>Gazebo/Grey</material>
   </gazebo>
   <!-- Attach the robotiq 85 gripper -->
@@ -41,6 +41,6 @@
     <origin xyz="0 0 0.004" rpy="0 ${-pi/2} ${pi}"/>
   </xacro:robotiq_85_gripper>
-  <xacro:robotiq_85_gripper_transmission prefix="" />
-  <xacro:ur_arm_transmission prefix="" />
+  <!-- <xacro:robotiq_85_gripper_transmission prefix="" /> -->
+  <!-- <xacro:ur_arm_transmission prefix="" /> -->
   <!-- Gazebo FT sensor plugin -->
   <gazebo reference="wrist_3_joint">
@@ -59,6 +59,6 @@
     <gripper name="gazebo_gripper">
       <grasp_check>
-        <attach_steps>2</attach_steps>    <!-- default: 20 -->
-        <detach_steps>2</detach_steps>    <!-- default: 40 -->
+        <attach_steps>20</attach_steps>    <!-- default: 20 -->
+        <detach_steps>40</detach_steps>    <!-- default: 40 -->
         <min_contact_count>3</min_contact_count>
       </grasp_check>
