Commit message: Added plugins and modified the params for better Gazebo simulation

File: src/robotiq_85/robotiq_description/urdf/robotiq_85_gripper.transmission.xacro (robot description, xacro)
@@ -19,5 +19,5 @@
                 <multiplier>1.0</multiplier>
                 <offset>0.0</offset>
-                <maxEffort>1000</maxEffort> <!-- This is crucial -->
+                <maxEffort>10000</maxEffort> <!-- This is crucial -->
                 <hasPID/> <!-- This is crucial -->
             </plugin>
@@ -27,5 +27,5 @@
                 <multiplier>1.0</multiplier>
                 <offset>0.0</offset>
-                <maxEffort>0.1</maxEffort> <!-- This is crucial -->
+                <maxEffort>10000</maxEffort> <!-- This is crucial -->
                 <hasPID/> <!-- This is crucial -->
             </plugin>
@@ -35,5 +35,5 @@
                 <multiplier>1.0</multiplier>
                 <offset>0.0</offset>
-                <maxEffort>0.1</maxEffort> <!-- This is crucial -->
+                <maxEffort>10000</maxEffort> <!-- This is crucial -->
                 <hasPID/> <!-- This is crucial -->
             </plugin>
@@ -43,5 +43,5 @@
                 <multiplier>-1.0</multiplier>
                 <offset>0.0</offset>
-                <maxEffort>0.1</maxEffort> <!-- This is crucial -->
+                <maxEffort>1000.0</maxEffort> <!-- This is crucial -->
                 <hasPID/> <!-- This is crucial -->
             </plugin>
@@ -51,25 +51,33 @@
                 <multiplier>-1.0</multiplier>
                 <offset>0.0</offset>
-                <maxEffort>0.1</maxEffort> <!-- This is crucial -->
+                <maxEffort>1000.0</maxEffort> <!-- This is crucial -->
                 <hasPID/> <!-- This is crucial -->
             </plugin>
-            <!-- This plugin fixes the problem when the object slips from the gripper
-                by "fixing" the object to the gripper
-            -->
-            <!-- <plugin name="gazebo_grasp_fix" filename="libgazebo_grasp_fix.so">
+        </gazebo>
+        <!-- This plugin fixes the problem when the object slips from the gripper
+        by "fixing" the object to the gripper -->
+        <gazebo>
+            <plugin name="gazebo_grasp_fix" filename="libgazebo_grasp_fix.so">
                 <arm>
-                    <arm_name>robotiq_85_gripper</arm_name>
-                    <palm_link>${prefix}robotiq_85_base_link</palm_link>
-                    <gripper_link> ${prefix}robotiq_85_left_knuckle_link </gripper_link>
+                    <arm_name>ur5</arm_name>
+                    <palm_link>${prefix}robotiq_85_left_knuckle_link</palm_link>
+                    <palm_link>${prefix}robotiq_85_right_knuckle_link</palm_link>
+                    <palm_link>${prefix}robotiq_85_left_inner_knuckle_link</palm_link>
+                    <palm_link>${prefix}robotiq_85_right_inner_knuckle_link</palm_link>
+                    <gripper_link> ${prefix}robotiq_85_right_finger_tip_link </gripper_link>
+                    <gripper_link> ${prefix}robotiq_85_left_finger_tip_link </gripper_link>
+                    <!-- <gripper_link> ${prefix}robotiq_85_left_knuckle_link </gripper_link>
                     <gripper_link> ${prefix}robotiq_85_right_knuckle_link </gripper_link>
+                    <gripper_link> ${prefix}robotiq_85_left_inner_knuckle_link </gripper_link>
+                    <gripper_link> ${prefix}robotiq_85_right_inner_knuckle_link </gripper_link> -->
                 </arm>
-                <forces_angle_tolerance>100</forces_angle_tolerance>
-                <update_rate>10</update_rate>
-                <grip_count_threshold>3</grip_count_threshold>
-                <max_grip_count>10</max_grip_count>
+                <forces_angle_tolerance>90</forces_angle_tolerance>
+                <update_rate>40</update_rate>
+                <grip_count_threshold>1</grip_count_threshold>
+                <max_grip_count>1</max_grip_count>
                 <release_tolerance>0.001</release_tolerance>
                 <disable_collisions_on_attach>false</disable_collisions_on_attach>
                 <contact_topic>__default_topic__</contact_topic>
-            </plugin> -->
+            </plugin>
         </gazebo>
     </xacro:macro>

File: src/robotiq_85/robotiq_description/urdf/robotiq_85_gripper.urdf.xacro (robot description, xacro)
@@ -33,12 +33,12 @@
       <axis xyz="0 0 1"/>
       <origin rpy="${pi} 0.0 0.0" xyz="0.05490451627 0.03060114443 0.0"/>
+      <limit lower="0.0" upper="0.80285" velocity="0.5" effort="10000"/>
+    </joint>
+    <joint name="${prefix}robotiq_85_right_knuckle_joint" type="continuous">
+      <parent link="${prefix}robotiq_85_base_link"/>
+      <child link="${prefix}robotiq_85_right_knuckle_link"/>
+      <axis xyz="0 0 1"/>
+      <origin rpy="0.0 0.0 0.0" xyz="0.05490451627 -0.03060114443 0.0"/>
       <limit lower="0.0" upper="0.80285" velocity="0.5" effort="1000"/>
-    </joint>
-    <joint name="${prefix}robotiq_85_right_knuckle_joint" type="continuous">
-      <parent link="${prefix}robotiq_85_base_link"/>
-      <child link="${prefix}robotiq_85_right_knuckle_link"/>
-      <axis xyz="0 0 1"/>
-      <origin rpy="0.0 0.0 0.0" xyz="0.05490451627 -0.03060114443 0.0"/>
-      <limit lower="-3.14" upper="3.14" velocity="100.0" effort="1000"/>
       <!-- <mimic joint="${prefix}robotiq_85_left_knuckle_joint"/> -->
     </joint>
@@ -239,16 +239,16 @@
     <!-- Improve grasping physics -->
     <gazebo reference="${prefix}robotiq_85_left_finger_tip_link">
-      <kp>10000000.0</kp>
-      <kd>1000.0</kd>
-      <mu1>10000.0</mu1>
-      <mu2>10000.0</mu2>
+      <kp>1000000000.0</kp>
+      <kd>1.0</kd>
+      <mu1>1.0</mu1>
+      <mu2>1.0</mu2>
       <maxVel>1.0</maxVel>
       <minDepth>0.001</minDepth>
     </gazebo>
     <gazebo reference="${prefix}robotiq_85_right_finger_tip_link">
-      <kp>10000000.0</kp>
-      <kd>1000.0</kd>
-      <mu1>10000.0</mu1>
-      <mu2>10000.0</mu2>
+      <kp>1000000000.0</kp>
+      <kd>1.0</kd>
+      <mu1>1.0</mu1>
+      <mu2>1.0</mu2>
       <maxVel>1.0</maxVel>
       <minDepth>0.001</minDepth>

File: src/ur5/ur5_description/urdf/ur5_robotiq85_gripper.urdf.xacro (robot description, xacro)
@@ -56,9 +56,9 @@
   </gazebo>
   <!-- Gazebo grasping plugin -->
-  <gazebo>
+  <!-- <gazebo>
     <gripper name="gazebo_gripper">
       <grasp_check>
-        <attach_steps>20</attach_steps>    <!-- default: 20 -->
-        <detach_steps>40</detach_steps>    <!-- default: 40 -->
+        <attach_steps>20</attach_steps>
+        <detach_steps>40</detach_steps>
         <min_contact_count>3</min_contact_count>
       </grasp_check>
@@ -67,5 +67,5 @@
       <palm_link>robotiq_85_base_link</palm_link>
     </gripper>
-  </gazebo>
+  </gazebo> -->
   <!-- Load gazebo_ros_control -->
   <xacro:include filename="$(find ur5_description)/urdf/common.gazebo.xacro" />
